File: src/HardwareDesign/DataForge-DAQ.sch (EAGLE design)
At the start: 64 parts, among them IC1 RP2354B, J1 HX TYPE-C 16PIN, X4 ABM8-272-T3

Commit message: review AIN
Parts:
- removed X3: (no value), con-subd:F37V
- removed X4: ABM8-272-T3, ds_passive:CRYSTAL
- added C21, C22: 18pF, ds_passive:C0402
- added C23, C24, C42, C43: 270pF, ds_passive:C0402
- added C25, C26, C27, C28, C29, C30, C31, C32, C33, C34, C35, C36, C37, C38, C39, C40, C51, C53, C55, C57, C59, C61, C63, C65, C67, C69, C71, C73: 100nF, ds_passive:C0603
- added C41, C44: 680pF, ds_passive:C0402
- added C45, C46, C49, C75, C76: 100nF, ds_passive:C0402
- added C47: 10uF, ds_passive:C0805
- added C48, C74: (no value), ds_passive:C0805
- added C50, C52, C54, C56, C58, C60, C62, C64, C66, C68, C70, C72: 1uF, ds_passive:C0603
- added IC10, IC11: MCP6001RT, ds_ic_opa:MCP6001RT
- added IC4: ADS1256, ds_ic_peripherals:ADS1256IDB
- added IC5, IC7: DG409, ds_ic_peripherals:DG409
- added IC6, IC8: ADA4254ACPZ, ds_ic_opa:ADA4254ACPZ
- added IC9: REF3025, maxim:MAX6520
- added J2, J3: (no value), con-subd:F37V
- added L2: BLM18RK102N1, ds_passive:R0805
- added R15, R18, R50: 100R, ds_passive:R0402
- added R16, R17: 10K, ds_passive:R0402
- added R19: CRA034RF100RP05Z, Resistor Array:YC164-JR-0733RL
- added R20, R21, R22, R23: 200R, ds_passive:R0402
- added R24, R42, R43, R44, R45, R46, R47, R48, R51, R52: 0R, ds_passive:R0603
- added R25, R26, R27, R28, R29, R30, R31, R32, R33, R34, R35, R36, R37, R38, R40, R41: 1K, ds_passive:R0603
- added R49: 20K, pot:TRIM_EU-3223G
- added TP17, TP18, TP19, TP20, TP21, TP22, TP23, TP24, TP25, TP26, TP27, TP28, TP29, TP30, TP31, TP32, TP33, TP34, TP35, TP36, TP37, TP38, TP39, TP40: PTR1B1,27, testpad:PTR1B1,27
- added USB: HX TYPE-C 16PIN, SparkFun-Connectors:USB_C_2-LAYER_PADS
- J1: value HX TYPE-C 16PIN -> (none); device SparkFun-Connectors:USB_C_2-LAYER_PADS -> con-subd:F37V
- X1: value (none) -> ABM8-272-T3; device con-subd:F37V -> ds_passive:CRYSTAL
- X2: value (none) -> 7.68MHz; device con-subd:F37V -> ds_passive:CRYSTAL
Connections:
- removed net AI_0: X2.3
- removed net AI_1: X2.22
- removed net AI_10: X2.8
- removed net AI_11: X2.27
- removed net AI_12: X2.9
- removed net AI_13: X2.28
- removed net AI_14: X2.10
- removed net AI_15: X2.29
- removed net AI_2: X2.4
- removed net AI_3: X2.23
- removed net AI_4: X2.5
- removed net AI_5: X2.24
- removed net AI_6: X2.6
- removed net AI_7: X2.25
- removed net AI_8: X2.7
- removed net AI_9: X2.26
- new net !ADC_PDWN: R17.2, R18.1
- new net !ADC_RST: R15.1, R16.2
- new net !CS1_ADC: IC4.!CS
- new net !CS_ADA_A: IC6.!CS
- new net !CS_ADA_B: IC8.!CS
- new net !DRDY: IC4.!DRDY
- new net +5V_A: IC4.AVDD, L2.2
- new net ADA_A_IO0: IC5.A0, IC6.GPIO0
- new net ADA_A_IO1: IC5.A1, IC6.GPIO1
- new net ADA_A_IO2: IC5.EN, IC6.GPIO2
- new net ADA_B_IO0: IC7.A0, IC8.GPIO0
- new net ADA_B_IO1: IC7.A1, IC8.GPIO1
- new net ADA_B_IO2: IC7.EN, IC8.GPIO2
- new net ADC_AIN_N: C24.2, C41.2, R21.1, R46.1, TP22.TP
- new net ADC_AIN_P: C23.1, C41.1, R20.1, R45.2, TP21.TP
- new net ADC_BIN_N: C43.2, C44.2, R23.1, R48.2, TP24.TP
- new net ADC_BIN_P: C42.1, C44.1, R22.1, R47.1, TP23.TP
- new net ADC_IN0: IC4.AI0, R45.1, TP17.TP
- new net ADC_IN1: IC4.AI1, R46.2, TP18.TP
- new net ADC_IN2: IC4.AI2, R48.1, TP19.TP
- new net ADC_IN3: IC4.AI3, R47.2, TP20.TP
- new net AI_0+: J2.3, R25.1
- new net AI_1-: J2.22, R26.1
- new net AI_10+: J2.8, R35.1
- new net AI_11-: J2.27, R36.1
- new net AI_12+: J2.9, R37.1
- new net AI_13-: J2.28, R38.1
- new net AI_14+: J2.10, R40.1
- new net AI_15-: J2.29, R41.1
- new net AI_2+: J2.4, R27.1
- new net AI_3-: J2.23, R28.1
- new net AI_4+: J2.5, R29.1
- new net AI_5-: J2.24, R30.1
- new net AI_6+: J2.6, R31.1
- new net AI_7-: J2.25, R32.1
- new net AI_8+: J2.7, R33.1
- new net AI_9-: J2.26, R34.1
- new net IN0+: C25.1, IC5.IN_A_0, R25.2
- new net IN1-: C26.1, IC5.IN_B_0, R26.2
- new net IN10+: C35.1, IC7.IN_A_1, R35.2
- new net IN11-: C36.1, IC7.IN_B_1, R36.2
- new net IN12+: C37.1, IC7.IN_A_2, R37.2
- new net IN13-: C38.1, IC7.IN_B_2, R38.2
- new net IN14+: C39.1, IC7.IN_A_3, R40.2
- new net IN15-: C40.1, IC7.IN_B_3, R41.2
- new net IN2+: C27.1, IC5.IN_A_1, R27.2
- new net IN3-: C28.1, IC5.IN_B_1, R28.2
- new net IN4+: C29.1, IC5.IN_A_2, R29.2
- new net IN5-: C30.1, IC5.IN_B_2, R30.2
- new net IN6+: C31.1, IC5.IN_A_3, R31.2
- new net IN7-: C32.1, IC5.IN_B_3, R32.2
- new net IN8+: C33.1, IC7.IN_A_0, R33.2
- new net IN9-: C34.1, IC7.IN_B_0, R34.2
- new net MISO: IC4.DOUT, IC6.SDO, IC8.SDO, R19.2
- new net MOSI: IC4.DIN, IC6.SDI, IC8.SDI, R19.3
- new net MUX_A_OUTA: IC5.OUT_A, R43.2, TP33.TP
- new net MUX_A_OUTB: IC5.OUT_B, R44.1, TP34.TP
- new net MUX_B_OUTA: IC7.OUT_A, R24.2, TP35.TP
- new net MUX_B_OUTB: IC7.OUT_B, R42.1, TP36.TP
- new net N$10: IC6.OUT-, R21.2
- new net N$11: IC11.+IN, R50.2
- new net N$15: IC8.OUT+, R22.2
- new net N$16: IC8.OUT-, R23.2
- new net N$22: TP28.TP
- new net N$33: TP39.TP
- new net N$34: TP40.TP
- new net N$5: IC4.!RESET, R15.2
- new net N$6: C74.1, R49.S, R50.1
- new net N$7: C72.2, C73.2, R49.A
- new net N$8: IC4.SYNC/PDOWN, R18.2
- new net N$9: IC6.OUT+, R20.2
- new net PGA_A_IN+: IC6.IN1+, R43.1, TP29.TP
- new net PGA_A_IN-: IC6.IN1-, IC6.IN2+, R44.2, TP30.TP
- new net PGA_B_IN+: IC8.IN1+, R24.1, TP31.TP
- new net PGA_B_IN-: IC8.IN1-, IC8.IN2+, R42.2, TP32.TP
- new net SCK: IC4.SCLK, IC6.SCK, IC8.SCK, R19.4
- new net SPI_MISO: R19.7
- new net SPI_MOSI: R19.6
- new net SPI_SCK: R19.5
- new net V+: C52.1, C53.1, C56.1, C57.1, C60.1, C61.1, C66.1, C67.1, IC5.V+, IC6.VDDH, IC7.V+, IC8.VDDH
- new net V-: C54.1, C55.1, C58.1, C59.1, C62.1, C63.1, C68.1, C69.1, IC5.V-, IC6.PAD, IC6.VSSH, IC7.V-, IC8.PAD, IC8.VSSH
- new net VOCM_A: IC6.VOCM, R51.2, TP37.TP
- new net VOCM_B: IC8.VOCM, R52.1, TP38.TP
- new net VREF: C46.1, C72.1, C73.1, IC10.-IN, IC10.OUT, IC4.AI4, IC4.VREFP, IC6.AVDD, IC8.AVDD, R49.E, TP25.TP
- new net VREF/2: C75.1, IC11.-IN, IC11.OUT, R51.1, R52.2, TP27.TP
- new net VREF_RAW: C48.1, IC10.+IN, IC9.OUT, TP26.TP
- new net XTAL1: C21.1, IC4.XTAL1, X2.CON
- new net XTAL2: C22.1, IC4.XTAL2, X2.OUT
- net +3V3: now also C45.1, C47.1, C49.1, C50.1, C51.1, C64.1, C65.1, C70.1, C71.1, C76.1, IC10.V+, IC11.V+, IC4.DVDD, IC6.DVDD, IC8.DVDD, IC9.IN, J1.19, J2.19, J3.19, J3.37, R16.1, R17.1; no longer X1.19, X2.19, X3.19, X3.37
- net +5V: now also J1.1, J1.20, J2.1, J2.20, J3.1, J3.20, L2.1; no longer X1.1, X1.20, X2.1, X2.20, X3.1, X3.20
- net AO_0: now also J2.12; no longer X2.12
- net AO_1: now also J2.31; no longer X2.31
- net AO_2: now also J2.13; no longer X2.13
- net AO_3: now also J2.32; no longer X2.32
- net AO_4: now also J2.14; no longer X2.14
- net AO_5: now also J2.33; no longer X2.33
- net AO_6: now also J2.15; no longer X2.15
- net AO_7: now also J2.34; no longer X2.34
- net CAN_H: now also J3.10; no longer X3.10
- net CAN_L: now also J3.29; no longer X3.29
- net CC1: now also USB.CC1; no longer J1.CC1
- net CC2: now also USB.CC2; no longer J1.CC2
- net DIO_0: now also J1.3; no longer X1.3
- net DIO_1: now also J1.22; no longer X1.22
- net DIO_10: now also J1.8; no longer X1.8
- net DIO_11: now also J1.27; no longer X1.27
- net DIO_12: now also J1.9; no longer X1.9
- net DIO_13: now also J1.28; no longer X1.28
- net DIO_14: now also J1.10; no longer X1.10
- net DIO_15: now also J1.29; no longer X1.29
- net DIO_16: now also J1.11; no longer X1.11
- net DIO_17: now also J1.30; no longer X1.30
- net DIO_18: now also J1.12; no longer X1.12
- net DIO_19: now also J1.31; no longer X1.31
- net DIO_2: now also J1.4; no longer X1.4
- net DIO_20: now also J1.13; no longer X1.13
- net DIO_21: now also J1.32; no longer X1.32
- net DIO_22: now also J1.14; no longer X1.14
- net DIO_23: now also J1.33; no longer X1.33
- net DIO_24: now also J1.15; no longer X1.15
- net DIO_25: now also J1.34; no longer X1.34
- net DIO_26: now also J1.16; no longer X1.16
- net DIO_27: now also J1.35; no longer X1.35
- net DIO_28: now also J1.17; no longer X1.17
- net DIO_29: now also J1.36; no longer X1.36
- net DIO_3: now also J1.23; no longer X1.23
- net DIO_30: now also J1.18; no longer X1.18
- net DIO_31: now also J1.37; no longer X1.37
- net DIO_4: now also J1.5; no longer X1.5
- net DIO_5: now also J1.24; no longer X1.24
- net DIO_6: now also J1.6; no longer X1.6
- net DIO_7: now also J1.25; no longer X1.25
- net DIO_8: now also J1.7; no longer X1.7
- net DIO_9: now also J1.26; no longer X1.26
- net D_N: now also USB.D-; no longer J1.D-
- net D_P: now also USB.D+; no longer J1.D+
- net GND: now also C21.2, C22.2, C23.2, C24.1, C25.2, C26.2, C27.2, C28.2, C29.2, C30.2, C31.2, C32.2, C33.2, C34.2, C35.2, C36.2, C37.2, C38.2, C39.2, C40.2, C42.2, C43.1, C45.2, C46.2, C47.2, C48.2, C49.2, C50.2, C51.2, C52.2, C53.2, C54.2, C55.2, C56.2, C57.2, C58.2, C59.2, C60.2, C61.2, C62.2, C63.2, C64.2, C65.2, C66.2, C67.2, C68.2, C69.2, C70.2, C71.2, C74.2, C75.2, C76.2, IC10.V-, IC11.V-, IC4.AGND, IC4.AI7, IC4.AICOM, IC4.DGND, IC4.VREFN, IC5.GND, IC6.AVSS, IC6.DVSS, IC6.IN2-, IC6.IOUT_HV, IC6.IOUT_LV, IC7.GND, IC8.AVSS, IC8.DVSS, IC8.IN2-, IC8.IOUT_HV, IC8.IOUT_LV, IC9.GND, J1.2, J1.21, J2.11, J2.2, J2.21, J2.30, J3.11, J3.15, J3.18, J3.2, J3.21, J3.26, J3.28, J3.30, J3.34, J3.36, J3.6, J3.7, J3.9, USB.GND, X1.VDD, X1.VSS, X2.VDD, X2.VSS; no longer J1.GND, X1.2, X1.21, X2.11, X2.2, X2.21, X2.30, X3.11, X3.15, X3.18, X3.2, X3.21, X3.26, X3.28, X3.30, X3.34, X3.36, X3.6, X3.7, X3.9, X4.VDD, X4.VSS
- net I2C_SCL: now also J3.35; no longer X3.35
- net I2C_SDA: now also J3.16; no longer X3.16
- net N$3: now also J3.17; no longer X3.17
- net QSPI_CLK: now also J3.14; no longer X3.14
- net QSPI_CS: now also J3.33; no longer X3.33
- net QSPI_D0: now also J3.12; no longer X3.12
- net QSPI_D1: now also J3.31; no longer X3.31
- net QSPI_D2: now also J3.13; no longer X3.13
- net QSPI_D3: now also J3.32; no longer X3.32
- net SHIELD: now also USB.SHLD; no longer J1.SHLD
- net UART0_CTS: now also J3.5; no longer X3.5
- net UART0_DCD: now also J3.25; no longer X3.25
- net UART0_DSR: now also J3.23; no longer X3.23
- net UART0_DTR: now also J3.4; no longer X3.4
- net UART0_RTS: now also J3.24; no longer X3.24
- net UART0_RX: now also J3.22; no longer X3.22
- net UART0_TX: now also J3.3; no longer X3.3
- net UART1_RX: now also J3.27; no longer X3.27
- net UART1_TX: now also J3.8; no longer X3.8
- net VBUS: now also USB.VBUS; no longer J1.VBUS
- net XIN: now also X1.CON; no longer X4.CON
- net XOUTC: now also X1.OUT; no longer X4.OUT
Other:
- note added: "+/-15V"
- note added: "0 0 1 OUT0"
- note added: "0 1 1 OUT1"
- note added: "1 0 1 OUT2"
- note added: "1 1 1 OUT3"
- note added: "1.25V"
- note added: "1.8V"
- note added: "2.5V"
- note added: "24 BIT ADC"
- note added: "3.3V"
- note added: "5V"
- note added: "A1 A0 EN ON"
- note added: "ADC INPUTS"
- note added: "ADS1256 ADC"
- note added: "ANALOG IN"
- note added: "ANALOG INPUT MUX"
- note added: "ANALOG OUTPUT"
- note added: "ANALOG-IN TESTPOINTS"
- note added: "BLOCK DIAGRAM"
- note added: "BOOST INVERTER TPS65131"
- note added: "CON1 DIO"
- note added: "CON2 AI AO"
- note added: "CON3 INTERFACING"
- note added: "DUAL LDO TPS7A39"
- note added: "IN0+ AND IN1-"
- note added: "IN10+ AND IN11-"
- note added: "IN12+ AND IN13-"
- note added: "IN14+ AND IN15-"
- note added: "IN2+ AND IN3-"
- note added: "IN4+ AND IN5-"
- note added: "IN6+ AND IN7-"
- note added: "IN8+ AND IN9-"
- note added: "INPUT MULTIPLEXER"
- note added: "LDO"
- note added: "MCU"
- note added: "PGA"
- note added: "POWER DELIVERY"
- note added: "REF"
- note added: "REF/2"
- note added: "V+ +12V"
- note added: "V- -12V"
- note added: "VOLTAGE REFERENCE"
- note added: "X X 0 -"
