File: src/HardwareDesign/DataForge-DAQ.sch (EAGLE design)
At the start: 281 parts, among them IC1 RP2354B, IC10 MCP6001RT, IC11 MCP6001RT, IC12 CYPD3177, IC13 INA180A3, IC14 TPS65131, IC15 TPS7A39, IC4 ADS1256, IC5 DG409, IC6 ADA4254ACPZ, IC7 DG409, IC8 ADA4254ACPZ, IC9 REF3025, Q1 2N7002, T1 DMP3098LSD, T2 IRLML5203, X1 ABM8-272-T3, X2 7.68MHz

Commit message: add new ADC
Parts:
- removed L2: BLM18RK102N1, ds_passive:R0805
- removed X2: 7.68MHz, ds_passive:CRYSTAL
- added C110: 10uF, ds_passive:C0805
- added C111: 100nF, ds_passive:C0603
- added C112, C113: 100nF, ds_passive:C0402
- added IC16, IC17: (no value), ds_ic_logic:74LVC08A
- added IC18: 74LVC32A, ds_ic_logic:74LVC32A
- added IC19: 74AHC1G04DBV, 74xx-little-us:74AHC1G04DBV
- added R81, R82, R83, R84, R85: 0R, ds_passive:R0402
- added TP52, TP58, TP59, TP60, TP61, TP62, TP63, TP64, TP65, TP66, TP67, TP68, TP69, TP70, TP71, TP72, TP73, TP74, TP75, TP76, TP77, TP78, TP79, TP80, TP81, TP82, TP83, TP84, TP85: PTR1B1,27, testpad:PTR1B1,27
- C21, C22: value 18pF -> 100nF
- C70: value 1uF -> 10uF; device ds_passive:C0603 -> ds_passive:C0805
- IC4: value ADS1256 -> ADS9234RIRHBR; device ds_ic_peripherals:ADS1256IDB -> ds_ic_peripherals:ADS9234RIRHBR
- R15, R18: value 100R -> 0R
- R17: value 10K -> 0R
Connections:
- removed net !ADC_PDWN: R17.2, R18.1
- removed net !DRDY: IC4.!DRDY
- removed net +5V_A: IC4.AVDD, L2.2
- removed net N$22: TP28.TP
- removed net N$33: TP39.TP
- removed net N$34: TP40.TP
- removed net XTAL1: C21.1, IC4.XTAL1, X2.CON
- removed net XTAL2: C22.1, IC4.XTAL2, X2.OUT
- new net !QSPI_SEL: IC17G$1.B, IC17G$2.B, IC17G$3.B, IC17G$4.B, IC19A.O, TP71.TP
- new net ADC_RDY: IC1.GPIO1, IC4.READY/STROBE, TP28.TP
- new net N$45: IC1.GPIO14, R83.2
- new net N$46: IC17G$1.Y, IC18G$1.B
- new net N$47: IC16G$2.Y, IC18G$2.A
- new net N$48: IC17G$2.Y, IC18G$2.B
- new net N$49: IC16G$3.Y, IC18G$3.A
- new net N$50: IC1.GPIO15, R84.2
- new net N$51: IC17G$3.Y, IC18G$3.B
- new net N$52: IC16G$4.Y, IC18G$4.A
- new net N$53: IC17G$4.Y, IC18G$4.B
- new net N$54: IC1.GPIO16, R85.2
- new net N$55: TP79.TP
- new net N$56: TP78.TP
- new net N$57: TP77.TP
- new net QSPI_SEL: IC1.GPIO3, IC16G$1.B, IC16G$2.B, IC16G$3.B, IC16G$4.B, IC19A.I, TP70.TP
- new net REFBY2: C71.1, IC4.REFBY2, TP85.TP
- new net REFM_A: C70.2, IC4.REFM_A, TP81.TP
- new net REFM_B: C110.2, IC4.REFM_B, TP83.TP
- new net REFOUT: C111.1, IC4.REFOUT, TP84.TP
- new net REFP_A: C70.1, IC4.REFP_A, TP80.TP
- new net REFP_B: C110.1, IC4.REFP_B, TP82.TP
- new net SDO_A_0: IC16G$1.A, IC4.SDO-0/0A, R17.2, TP62.TP
- new net SDO_A_1: IC16G$2.A, IC4.SDO-1/1A, R18.2, TP63.TP
- new net SDO_A_2: IC16G$3.A, IC4.SDO-2/2A, R81.2, TP64.TP
- new net SDO_A_3: IC16G$4.A, IC4.SDO-3/3A, R82.2, TP65.TP
- new net SDO_B_0: IC17G$1.A, IC4.SDO-4/0B, R17.1, TP66.TP
- new net SDO_B_1: IC17G$2.A, IC4.SDO-5/1B, R18.1, TP67.TP
- new net SDO_B_2: IC17G$3.A, IC4.SDO-6/2B, R81.1, TP68.TP
- new net SDO_B_3: IC17G$4.A, IC4.SDO-7/3B, R82.1, TP69.TP
- net !ADC_RST: now also IC1.GPIO2, IC4.!PD!/!RST, TP39.TP; no longer R15.1
- net !CS1_ADC: now also IC1.GPIO9, R15.1, TP40.TP
- net !CS_ADA_B: now also IC1.GPIO7
- net +3V3: now also C112.1, C113.1, C21.1, C22.1, IC16G$5.VCC, IC17G$5.VCC, IC18G$5.VCC, IC19P.VCC, IC4.AVDD; no longer C70.1, C71.1, R17.1
- net +5V: no longer L2.1
- net ADA_B_IO0: now also R83.1
- net ADA_B_IO1: now also R84.1
- net ADA_B_IO2: now also R85.1
- net ADC_IN0: now also IC4.AINP_A; no longer IC4.AI0
- net ADC_IN1: now also IC4.AINM_A; no longer IC4.AI1
- net ADC_IN2: now also IC4.AINP_B; no longer IC4.AI2
- net ADC_IN3: now also IC4.AINM_B; no longer IC4.AI3
- net GND: now also C111.2, C112.2, C113.2, IC16G$5.GND, IC17G$5.GND, IC18G$5.GND, IC19P.GND, IC4.GND, IC4.PAD; no longer C70.2, IC4.AGND, IC4.AI7, IC4.AICOM, IC4.DGND, IC4.VREFN, X2.VDD, X2.VSS
- net ISINK_COARSE: now also TP60.TP
- net ISINK_FINE: now also TP61.TP
- net MISO: now also IC1.GPIO8, TP73.TP; no longer IC4.DOUT
- net MOSI: now also IC1.GPIO11, IC4.SDI, TP72.TP; no longer IC4.DIN
- net N$5: now also IC4.CONVST; no longer IC4.!RESET
- net N$8: now also IC16G$1.Y, IC18G$1.A; no longer IC4.SYNC/PDOWN, R18.2
- net PDC_VCCD: now also TP52.TP
- net PD_FLIP: now also IC1.GPIO5
- net PD_GPIO: now also IC1.GPIO6
- net PD_INT: now also IC1.GPIO4
- net QSPI_SD0: now also IC18G$1.Y
- net QSPI_SD1: now also IC18G$2.Y
- net QSPI_SD2: now also IC18G$3.Y
- net QSPI_SD3: now also IC18G$4.Y
- net SCK: now also IC1.GPIO10, TP74.TP
- net SCL: now also IC1.GPIO13, TP76.TP
- net SDA: now also IC1.GPIO12, TP75.TP
- net USB_ISENSE: now also IC1.GPIO40_ADC0
- net VBUS_MAX: now also TP58.TP
- net VBUS_MIN: now also TP59.TP
- net VREF: no longer IC4.AI4, IC4.VREFP
Other:
- note added: "14 BIT ADC"
- note added: "3.3V SYTEM LDO"
- note added: "3.3V TARGET LDO"
- note added: "ADS9234R ADC"
- note added: "CYPD3177 POWER DELIVERY"
- note added: "PD CURRENT SENSOR"
- note added: "QSPI DATA LINE SELECT"
- note removed: "24 BIT ADC"
- note removed: "ADS1256 ADC"
- moved on the sheet: C1, C10, C11, C12, C13, C14, C15, C16, C17, C18, C19, C2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

Commit message: add DIO to design
Parts:
- removed J3: (no value), con-subd:F37V
- removed TP79: PTR1B1,27, testpad:PTR1B1,27
- added C114, C116, C120, C121, C125, C126, C128, C129, C131, C132, C134, C135, C137, C138, C140, C141, C143, C144, C146, C147, C149, C150: 100nF, ds_passive:C0402
- added C115, C117: 4.7uF, ds_passive:C0603
- added C118, C119: 100uF, rcl:CPOL-EU153CLV-0605
- added C122, C124, C151, C153, C155, C157, C159, C161, C163, C165, C167, C169: 1uF, ds_passive:C0603
- added C123, C152, C154, C156, C158, C160, C162, C164, C166, C168, C170, C171: 100nF, ds_passive:C0603
- added C127, C130, C133, C136, C139, C142, C145, C148: 20nF, ds_passive:C0402
- added IC20: MIC5504-3.3YM5-TR, ds_ic_vreg:MIC5504-3.3YM5-TR
- added IC21: LD117ADT33TR, v-reg:LD117ADT33TR
- added IC22: DAC8568, ds_ic_peripherals:DAC8568
- added IC23, IC24, IC25, IC26, IC27, IC28, IC29, IC30, IC31: MCP6001RT, ds_ic_opa:MCP6001RT
- added IC32, IC33, IC34, IC35: LSF0108, ds_ic_peripherals:LSF0108-Q1
- added IC36: MCP23S18, ds_ic_peripherals:MCP23S18
- added IC37: (no value), ds_ic_peripherals:MCP23S18
- added IC38: (no value), ds_ic_peripherals:SN74LVC2G66
- added IC39: 74LVC1G04, ds_ic_logic:74LVC1G04
- added R100, R103, R104, R107, R108, R111, R112, R115, R116, R87, R88, R91, R92, R95, R96, R99: 10K 0.1%, ds_passive:R0402
- added R101, R105, R109, R113, R117, R89, R93, R97: 43K 0.1%, ds_passive:R0402
- added R102, R106, R110, R114, R118, R90, R94, R98: 68R 1%, ds_passive:R0402
- added R119, R120, R121, R122, R123, R124, R125, R126: YC164-JR-0733RL, Resistor Array:YC164-JR-0733RL
- added R127, R128, R129, R130: 200K, ds_passive:R0402
- added R86: CRA034RF100RP05Z, Resistor Array:YC164-JR-0733RL
- added TP100, TP101, TP102, TP103, TP104, TP105, TP106, TP86, TP87, TP88, TP89, TP90, TP91, TP92, TP93, TP94, TP95, TP96, TP97, TP98, TP99: PTR1B1,27, testpad:PTR1B1,27
Connections:
- net VREF renamed VREF_ADC
- net VREF/2 renamed VREF_ADC/2
- net VREF_RAW renamed VREF_ADC_RAW
- removed net CAN_H: J3.10
- removed net CAN_L: J3.29
- removed net N$3: J3.17
- removed net N$55: TP79.TP
- removed net N$56: TP78.TP
- removed net N$57: TP77.TP
- removed net QSPI_CLK: J3.14
- removed net QSPI_CS: J3.33
- removed net QSPI_D0: J3.12
- removed net QSPI_D1: J3.31
- removed net QSPI_D2: J3.13
- removed net QSPI_D3: J3.32
- removed net UART0_DCD: J3.25
- removed net UART0_DSR: J3.23
- removed net UART0_DTR: J3.4
- new net !DIO_LEVEL_SELECT: IC38.2C, IC39.OUT
- new net DAC_!CLR: IC1.GPIO20, IC22.!CLR, R86.1, TP93.TP
- new net DAC_!LDAC: IC1.GPIO18, IC22.!LDAC, R86.3, TP89.TP
- new net DAC_!SYNC: IC1.GPIO19, IC22.!SYNC, R86.2, TP91.TP
- new net DAC_0: IC22.VOUT_A, IC24.+IN, TP90.TP
- new net DAC_1: IC22.VOUT_B, IC25.+IN, TP92.TP
- new net DAC_2: IC22.VOUT_C, IC26.+IN, TP94.TP
- new net DAC_3: IC22.VOUT_D, IC27.+IN, TP96.TP
- new net DAC_4: IC22.VOUT_E, IC28.+IN, TP97.TP
- new net DAC_5: IC22.VOUT_F, IC29.+IN, TP98.TP
- new net DAC_6: IC22.VOUT_G, IC30.+IN, TP99.TP
- new net DAC_7: IC22.VOUT_H, IC31.+IN, TP100.TP
- new net DIO_CS1: IC1.GPIO23, IC36.!CS, TP104.TP
- new net DIO_CS2: IC1.GPIO24, IC37.!CS
- new net DIO_EN: IC1.GPIO25, IC32.EN, IC33.EN, IC34.EN, IC35.EN, TP103.TP
- new net DIO_LEVEL_SELECT: IC1.GPIO26, IC38.1C, IC39.IN, TP101.TP, TP106.TP
- new net DIO_RESET: IC36.!RESET, IC37.!RESET, TP105.TP
- new net N$100: IC34.B1, R123.1
- new net N$101: IC34.B2, R123.2
- new net N$102: IC34.B3, R123.3
- new net N$103: IC34.B4, R123.4
- new net N$104: IC34.B5, R124.1
- new net N$105: IC34.B6, R124.2
- new net N$106: IC34.B7, R124.3
- new net N$107: IC34.B8, R124.4
- new net N$108: IC35.A3, IC37.GPB2
- new net N$109: IC35.A4, IC37.GPB3
- new net N$110: IC35.A5, IC37.GPB4
- new net N$111: IC35.A6, IC37.GPB5
- new net N$112: IC35.A7, IC37.GPB6
- new net N$113: IC35.A8, IC37.GPB7
- new net N$114: IC35.A2, IC37.GPB1
- new net N$115: IC35.A1, IC37.GPB0
- new net N$116: IC35.B1, R125.1
- new net N$117: IC35.B2, R125.2
- new net N$118: IC35.B3, R125.3
- new net N$119: IC35.B4, R125.4
- new net N$120: IC35.B5, R126.1
- new net N$121: IC35.B6, R126.2
- new net N$122: IC35.B7, R126.3
- new net N$123: IC35.B8, R126.4
- new net N$124: IC32.VREF_B, R127.1
- new net N$125: IC33.VREF_B, R128.1
- new net N$126: IC35.VREF_B, R129.1
- new net N$127: IC34.VREF_B, R130.1
- new net N$14: C129.2, IC24.OUT, R90.1
- new net N$17: C129.1, IC24.-IN, R87.2, R88.2, R89.1
- new net N$22: C132.1, IC25.-IN, R91.2, R92.2, R93.1
- new net N$23: C132.2, IC25.OUT, R94.1
- new net N$25: C135.1, IC26.-IN, R95.2, R96.2, R97.1
- new net N$26: C135.2, IC26.OUT, R98.1
- new net N$27: C138.1, IC27.-IN, R100.2, R101.1, R99.2
- new net N$28: C138.2, IC27.OUT, R102.1
- new net N$29: IC33.A2, IC36.GPB1
- new net N$31: C141.1, IC28.-IN, R103.2, R104.2, R105.1
- new net N$33: C141.2, IC28.OUT, R106.1
- new net N$34: C144.1, IC29.-IN, R107.2, R108.2, R109.1
- new net N$40: C144.2, IC29.OUT, R110.1
- new net N$41: C147.1, IC30.-IN, R111.2, R112.2, R113.1
- new net N$58: C147.2, IC30.OUT, R114.1
- new net N$59: C150.1, IC31.-IN, R115.2, R116.2, R117.1
- new net N$60: C150.2, IC31.OUT, R118.1
- new net N$61: IC32.A1, IC36.GPA0
- new net N$62: IC32.A2, IC36.GPA1
- new net N$63: IC32.A3, IC36.GPA2
- new net N$64: IC32.A4, IC36.GPA3
- new net N$65: IC32.A5, IC36.GPA4
- new net N$66: IC32.A6, IC36.GPA5
- new net N$67: IC32.A7, IC36.GPA6
- new net N$68: IC32.A8, IC36.GPA7
- new net N$69: IC32.B1, R119.1
- new net N$70: IC32.B2, R119.2
- new net N$71: IC32.B3, R119.3
- new net N$72: IC32.B4, R119.4
- new net N$73: IC32.B5, R120.1
- new net N$74: IC32.B6, R120.2
- new net N$75: IC32.B7, R120.3
- new net N$76: IC32.B8, R120.4
- new net N$77: IC33.A1, IC36.GPB0
- new net N$78: IC33.A3, IC36.GPB2
- new net N$79: IC33.A4, IC36.GPB3
- new net N$80: IC33.A5, IC36.GPB4
- new net N$81: IC33.A6, IC36.GPB5
- new net N$82: IC33.A7, IC36.GPB6
- new net N$83: IC33.A8, IC36.GPB7
- new net N$84: IC33.B1, R121.1
- new net N$85: IC33.B2, R121.2
- new net N$86: IC33.B3, R121.3
- new net N$87: IC33.B4, R121.4
- new net N$88: IC33.B5, R122.1
- new net N$89: IC33.B6, R122.2
- new net N$90: IC33.B7, R122.3
- new net N$91: IC33.B8, R122.4
- new net N$92: IC34.A1, IC37.GPA0
- new net N$93: IC34.A2, IC37.GPA1
- new net N$94: IC34.A3, IC37.GPA2
- new net N$95: IC34.A4, IC37.GPA3
- new net N$96: IC34.A5, IC37.GPA4
- new net N$97: IC34.A6, IC37.GPA5
- new net N$98: IC34.A7, IC37.GPA6
- new net N$99: IC34.A8, IC37.GPA7
- new net VREF_DAC: C125.1, IC23.-IN, IC23.OUT, R100.1, R104.1, R108.1, R112.1, R116.1, R88.1, R92.1, R96.1
- new net VREF_DAC_OUT: C124.1, IC22.VREF_IO, IC23.+IN, TP95.TP
- new net V_OUT_REF: C153.1, C154.1, C157.1, C158.1, C161.1, C162.1, C165.1, C166.1, IC38.1B, IC38.2B, R127.2, R128.2, R129.2, R130.2, TP102.TP
- net !CS1_ADC: now also IC1.GPIO21; no longer IC1.GPIO9
- net !CS_ADA_B: now also IC1.GPIO22; no longer IC1.GPIO7
- net +3V3: now also C116.1, C117.1, C122.1, C123.1, C126.1, C128.1, C131.1, C134.1, C137.1, C140.1, C143.1, C146.1, C149.1, C151.1, C152.1, C155.1, C156.1, C159.1, C160.1, C163.1, C164.1, C167.1, C168.1, C169.1, C170.1, C171.1, IC20.VOUT, IC22.AVDD, IC23.V+, IC24.V+, IC25.V+, IC26.V+, IC27.V+, IC28.V+, IC29.V+, IC30.V+, IC31.V+, IC32.VREF_A, IC33.VREF_A, IC34.VREF_A, IC35.VREF_A, IC36.VDD, IC37.VDD, IC38.1A, IC38.VCC, IC39.V+, R86.6, R86.7, R86.8, TP87.TP
- net +3V3_EXT: now also C119.+, C121.1, IC21.OUT, TP86.TP; no longer J3.19, J3.37
- net +5V: now also C114.1, C115.1, C118.+, C120.1, IC20.EN, IC20.VIN, IC21.IN, IC38.2A
- net +5V_EXT: no longer J3.1, J3.20
- net AO_0: now also C127.1, R89.2, R90.2
- net AO_1: now also C130.1, R93.2, R94.2
- net AO_2: now also C133.1, R97.2, R98.2
- net AO_3: now also C136.1, R101.2, R102.2
- net AO_4: now also C139.1, R105.2, R106.2
- net AO_5: now also C142.1, R109.2, R110.2
- net AO_6: now also C145.1, R113.2, R114.2
- net AO_7: now also C148.1, R117.2, R118.2
- net DIO_0: now also R119.8
- net DIO_1: now also R119.7
- net DIO_10: now also R121.6
- net DIO_11: now also R121.5
- net DIO_12: now also R122.8
- net DIO_13: now also R122.7
- net DIO_14: now also R122.6
- net DIO_15: now also R122.5
- net DIO_16: now also R123.8
- net DIO_17: now also R123.7
- net DIO_18: now also R123.6
- net DIO_19: now also R123.5
- net DIO_2: now also R119.6
- net DIO_20: now also R124.8
- net DIO_21: now also R124.7
- net DIO_22: now also R124.6
- net DIO_23: now also R124.5
- net DIO_24: now also R125.8
- net DIO_25: now also R125.7
- net DIO_26: now also R125.6
- net DIO_27: now also R125.5
- net DIO_28: now also R126.8
- net DIO_29: now also R126.7
- net DIO_3: now also R119.5
- net DIO_30: now also R126.6
- net DIO_31: now also R126.5
- net DIO_4: now also R120.8
- net DIO_5: now also R120.7
- net DIO_6: now also R120.6
- net DIO_7: now also R120.5
- net DIO_8: now also R121.8
- net DIO_9: now also R121.7
- net FLASH2_SS: now also TP78.TP
- net FLASH_SS: now also TP77.TP
- net GND: now also C114.2, C115.2, C116.2, C117.2, C118.-, C119.-, C120.2, C121.2, C122.2, C123.2, C124.2, C125.2, C126.2, C127.2, C128.2, C130.2, C131.2, C133.2, C134.2, C136.2, C137.2, C139.2, C140.2, C142.2, C143.2, C145.2, C146.2, C148.2, C149.2, C151.2, C152.2, C153.2, C154.2, C155.2, C156.2, C157.2, C158.2, C159.2, C160.2, C161.2, C162.2, C163.2, C164.2, C165.2, C166.2, C167.2, C168.2, C169.2, C170.2, C171.2, IC20.GND, IC21.ADJ, IC22.GND, IC23.V-, IC24.V-, IC25.V-, IC26.V-, IC27.V-, IC28.V-, IC29.V-, IC30.V-, IC31.V-, IC32.GND, IC33.GND, IC34.GND, IC35.GND, IC36.VSS, IC37.VSS, IC38.GND, IC39.V-, R103.1, R107.1, R111.1, R115.1, R87.1, R91.1, R95.1, R99.1, TP88.TP; no longer J3.11, J3.15, J3.18, J3.2, J3.21, J3.26, J3.28, J3.30, J3.34, J3.36, J3.6, J3.7, J3.9
- net I2C_SCL: now also IC1.GPIO29; no longer J3.35
- net I2C_SDA: now also IC1.GPIO28; no longer J3.16
- net MISO: now also IC36.SO, IC37.SO
- net MOSI: now also IC22.DIN, IC36.SI, IC37.SI
- net SCK: now also IC22.SCLK, IC36.SCK, IC37.SCK
- net UART0_CTS: now also IC1.GPIO30; no longer J3.5
- net UART0_RTS: now also IC1.GPIO31; no longer J3.24
- net UART0_RX: now also IC1.GPIO33; no longer J3.22
- net UART0_TX: now also IC1.GPIO32; no longer J3.3
- net UART1_RX: now also IC1.GPIO37; no longer J3.27
- net UART1_TX: now also IC1.GPIO36; no longer J3.8
Other:
- note added: "+/-12V POWER"
- note added: "16 BIT DAC 8 CHANNEL"
- note added: "2.5V VREF"
- note added: "ANALOG-OUT DAC"
- note added: "ANALOG-OUT OUTPUT DRIVERS"
- note added: "ANALOG-OUT TESTPOINTS"
- note added: "CON2 AI / AO"
- note added: "Choose R_ISOLATION = 68 Ω: 1. Stability with Capacitive Load: The combination of R_ISO and C_LOAD creates a low-pass filter. The cutoff frequency is: f_c = 1 / (2 * π * R_ISO * C_LOAD) For R_ISO = 68 Ω and C_LOAD = 20 nF: f_c = 1 / (2 * π * 68 * 20e-9) ≈ 117.2 kHz 2. Voltage Drop Across R_ISO: The voltage drop is: V_drop = I_load * R_ISO"
- note added: "DAC8568 Output Calculation: V_OUT = (1 + R_FB/R_G2 + R_FB/R_G1) * V_DAC - (R_FB/R_G2) * V_REF Given: Supply voltage: +/-12V Reference voltage (V_REF): 2.5V DAC resolution: 16 bits Desired output range: -12V to +12V 1. Determine the Gain (G): G = (V_OUT_max - V_OUT_min) / (V_DAC_max - V_DAC_min) G = (12 - (-12)) / (2.5 - 0) = 24 / 2.5 = 9.6 2. Solve for Resistor Ratios: G = 1 + R_FB/R_G2 + R_FB/R_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"
- note added: "DIGITAL IO"
- note added: "DIGITAL IO - LOWER 16 BITS"
- note added: "DIGITAL IO - UPPER 16 BITS"
- note added: "EXTTERNAL LDO"
- note added: "IO EXPANDER"
- note added: "LEVEL SELECTOR 3.3V/5V"
- note added: "OUTPUT DRIVERS"
- note added: "Sheet: Analog Input"
- note added: "Sheet: Analog Output"
- note added: "Sheet: Digital IO"
- note added: "Sheet: MCU"
- note added: "Sheet: Output Connectors"
- note added: "Sheet: POWER I."
- note added: "Sheet: POWER II."
- note added: "VOLTAGE LEVEL TRANSLATOR"
- note removed: "1.8V"
- note removed: "CON2 AI AO"
- note removed: "POWER"
- note removed: "VOLTAGE REFERENCE"
